File: fcBoard_Ethernet.kicad_sch (KiCad schematic)
At the start: 6 parts, among them J6 RJ45_MagJack, J7 RJ45_MagJack, U14 RTL8211F-CG, U15 RTL8211F-CG, Y1 25MHz, Y2 25MHz

Commit message: 회로도 라벨
Parts:
- renumbered J7 to J?, J6 to J?, U15 to U?, U14 to U?, Y1 to Y?, Y2 to Y?
Other:
- moved on the sheet: J?, U?, Y?
