File: fcBoard_Ethernet.kicad_sch (KiCad schematic)
At the start: 16 parts, among them J6 RJ45_MagJack, J7 RJ45_MagJack, U14 RTL8211F-CG, U15 RTL8211F-CG, Y1 25MHz, Y2 25MHz

Commit message: 11
Parts:
- removed C10, C6, C7, C9: 22pF, Capacitor_SMD:C_0402_1005Metric, symbol Device:C
- removed C5, C8: 100nF, Capacitor_SMD:C_0402_1005Metric, symbol Device:C
- removed FB1, FB2: 600R@100MHz, Inductor_SMD:L_0402_1005Metric, symbol Device:Ferrite_Bead
- removed J6, J7: RJ45_MagJack, Connector_RJ:RJ45_Amphenol_RJHSE538X_Horizontal, symbol Connector:RJ45_MagJack
- removed R8, R9: 4.7K, Resistor_SMD:R_0402_1005Metric, symbol Device:R
- removed U14, U15: RTL8211F-CG, Package_DFN_QFN:QFN-48-1EP_6x6mm_P0.4mm_EP4.25x4.25mm, symbol Interface_Ethernet:RTL8211F
- removed Y1, Y2: 25MHz, Crystal:Crystal_SMD_3215-2Pin_3.2x1.5mm, symbol Device:Crystal
- added J6, J7: RJ45_MagJack, Connector_RJ:RJ45_Amphenol_RJHSE538X_Horizontal, symbol RJ45_MagJack
- added U14, U15: RTL8211F-CG, Package_DFN_QFN:QFN-48-1EP_6x6mm_P0.4mm_EP4.25x4.25mm, symbol RTL8211F-CG
- added Y1, Y2: 25MHz, Crystal:Crystal_SMD_3215-2Pin_3.2x1.5mm, symbol Crystal
Connections:
- net GND: now also J6.13 (GND), J7.13 (GND), U14.24 (GND), U15.24 (GND)
Other:
- company: fcBoard Project -> fcBoard
- title: Gigabit Ethernet -> Dual Gigabit Ethernet

Commit message: 45
Parts:
- removed J7: RJ45_MagJack, Connector_RJ:RJ45_Amphenol_RJHSE538X_Horizontal, symbol RJ45_MagJack
- removed Y1, Y2: 25MHz, Crystal:Crystal_SMD_3215-2Pin_3.2x1.5mm, symbol Crystal
- added C301, C303, C305, C307, C309: 100nF, Capacitor_SMD:C_0402_1005Metric, symbol Device:C
- added C302, C304, C306, C308: 10uF, Capacitor_SMD:C_0603_1608Metric, symbol Device:C
- added R12, R13, R25: 10k, Resistor_SMD:R_0402_1005Metric, symbol Device:R
- J5: renamed from J6; footprint Connector_RJ:RJ45_Amphenol_RJHSE538X_Horizontal -> Connector_RJ:RJ45_Hanrun_HR911105A_Horizontal
- U11: renamed from U14; footprint Package_DFN_QFN:QFN-48-1EP_6x6mm_P0.4mm_EP4.25x4.25mm -> Package_DFN_QFN:QFN-48-1EP_7x7mm_P0.5mm_EP5.6x5.6mm
- U12: renamed from U15; footprint Package_DFN_QFN:QFN-48-1EP_6x6mm_P0.4mm_EP4.25x4.25mm -> Package_DFN_QFN:QFN-48-1EP_7x7mm_P0.5mm_EP5.6x5.6mm
Connections:
- net +3V3: now also R12.1, R13.1
- net ETH1_MDIO: now also R12.2
- net ETH2_MDIO: now also R13.2
- net GND: now also J5.SH (GND); no longer J5.13 (GND)
- net ETH2_PHYRST: now reaches U12.15 (TXP_A)
- net ETH1_PHYRST: now reaches U11.15 (TXP_A)
Other:
- note added: "MDIO Pullup Resistors 10kΩ for proper I2C-like bus operation"
- note added: "PHY Reset RC Circuit: R25=10kΩ, C309=100nF Provides ~10ms delay on power-up"
- note added: "RTL8211F U11 (ETH1) Decoupling: C301-C302: VDD33, C303-C304: VDD10 100nF + 10uF per rail"
- note added: "RTL8211F U12 (ETH2) Decoupling: C305-C306: VDD33, C307-C308: VDD10 100nF + 10uF per rail"
- moved on the sheet: J5
