File: fcBoard_Ethernet.kicad_sch (KiCad schematic)
At the start: 6 parts, among them J6 RJ45_MagJack, J7 RJ45_MagJack, U14 RTL8211F-CG, U15 RTL8211F-CG, Y1 25MHz, Y2 25MHz

Commit message: 45
Parts:
- removed J6, J7: RJ45_MagJack, Connector_RJ:RJ45_Amphenol_RJHSE538X_Horizontal, symbol RJ45_MagJack
- removed U14, U15: RTL8211F-CG, Package_DFN_QFN:QFN-48-1EP_6x6mm_P0.4mm_EP4.25x4.25mm, symbol RTL8211F-CG
- removed Y1, Y2: 25MHz, Crystal:Crystal_SMD_3215-2Pin_3.2x1.5mm, symbol Crystal
- added C14, C15, C22, C23: 22pF, jlc_components:C0402, symbol fcBoard:C
- added C16, C17, C19, C20: 100nF, jlc_components:C0402, symbol fcBoard:C
- added C18, C21: 1uF, jlc_components:C0603, symbol fcBoard:C
- added J6, J7: RJ45, jlc_components:RJ45-TH_8P8C_L21.0-W16.0-H13.0, symbol fcBoard:RJ45_Magjack
- added R8, R9: 10k, jlc_components:R0402, symbol fcBoard:R
- added U6, U7: RTL8211F-CG, Package_DFN_QFN:QFN-48-1EP_7x7mm_P0.5mm_EP5.3x5.3mm, symbol fcBoard:RTL8211F
- added Y2, Y3: 25MHz, jlc_components:HC-49S_L11.0-W4.6, symbol fcBoard:Crystal
Connections:
- net GND: now also U6.GND, U7.GND
- new net: C16.2, C17.1
- new net: C17.2, C18.1
- new net: C19.2, C20.1
- new net: C20.2, C21.1
Other:
- note added: "PL Gigabit Ethernet (ETH1) RGMII Interface"
- note added: "PS Gigabit Ethernet (ETH0) RGMII Interface"
- company: fcBoard -> fcBoard Project

Commit message: 자동화
Other:
- moved on the sheet: C14, C15, C16, C17, C18, C19, C20, C21, C22, C23, J6, J7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
