File: fcBoard_HDMI.kicad_sch (KiCad schematic)
At the start: 12 parts, among them J8 HDMI_IN, J9 HDMI_OUT, U16 TPD12S016, U17 IT6801FN, U18 TXB0108, U19 IT66121FN, U20 TPD12S016, Y3 27MHz, Y4 27MHz

Commit message: 회로도 라벨
Parts:
- renumbered C11 to C36, C12 to C37, J9 to J23, J8 to J24, R10 to R24, U19 to U41, U18 to U42, U17 to U43, U16 to U44, U20 to U45, Y3 to Y10, Y4 to Y9
