File: fcBoard_HDMI.kicad_sch (KiCad schematic)
At the start: 12 parts, among them J23 HDMI_OUT, J24 HDMI_IN, U41 IT66121FN, U42 TXB0108, U43 IT6801FN, U44 TPD12S016, U45 TPD12S016, Y10 27MHz, Y9 27MHz

Commit message: 45
Parts:
- removed C36, C37: 100nF, Capacitor_SMD:C_0402_1005Metric, symbol Device:C
- added C101, C102, C103, C104: 20pF, Capacitor_SMD:C_0402_1005Metric, symbol Device:C
- added C111, C113, C115, C121, C123, C125: 100nF, Capacitor_SMD:C_0402_1005Metric, symbol Device:C
- added C112, C114, C116, C122, C124, C126: 10uF, Capacitor_SMD:C_0603_1608Metric, symbol Device:C
- added R23: 4.7k, Resistor_SMD:R_0402_1005Metric, symbol Device:R
- added R26: 10k, Resistor_SMD:R_0402_1005Metric, symbol Device:R
- added R27: 27k, Resistor_SMD:R_0402_1005Metric, symbol Device:R
- J23, J24: footprint Connector_HDMI:HDMI_A_Molex_2086581051_Horizontal -> fcBoard_Connectors:HDMI_A_Contact_Technology_HDMI-19APL2_Horizontal
- R24: value 10K -> 4.7k
Connections:
- net GND: now also C101.2, C102.2, C103.2, C104.2
- net HDMI_I2C_SCL: now also R23.2
- net HDMI_I2C_SDA: now also R24.2
- net at R24.1: now also R23.1
Other:
- note added: "Crystal Load Capacitors Y9 (IT6801FN): C101, C102 = 20pF Y10 (IT66121FN): C103, C104 = 20pF"
- note added: "HDMI I2C Pullup Resistors 4.7kΩ for SCL and SDA"
- note added: "IT66121FN (HDMI TX) Decoupling: C121-C126: VDD33, VDD18, VDD12 100nF + 10uF per rail"
- note added: "IT6801FN (HDMI RX) Decoupling: C111-C116: VDD33, VDD18, VDD12 100nF + 10uF per rail"
