File: fcBoard_HDMI.kicad_sch (KiCad schematic)
At the start: 12 parts, among them J8 HDMI_IN, J9 HDMI_OUT, U16 TPD12S016, U17 IT6801FN, U18 TXB0108, U19 IT66121FN, U20 TPD12S016, Y3 27MHz, Y4 27MHz

Commit message: 45
Parts:
- removed C11, C12: 100nF, Capacitor_SMD:C_0402_1005Metric, symbol Device:C
- removed J8: HDMI_IN, Connector_HDMI:HDMI_A_Molex_2086581051_Horizontal, symbol Connector:HDMI_A
- removed J9: HDMI_OUT, Connector_HDMI:HDMI_A_Molex_2086581051_Horizontal, symbol Connector:HDMI_A
- removed R10: 10K, Resistor_SMD:R_0402_1005Metric, symbol Device:R
- removed U16, U20: TPD12S016, Package_DFN_QFN:QFN-24-1EP_4x4mm_P0.5mm_EP2.7x2.7mm, symbol Power_Protection:TPD12S016
- removed U17: IT6801FN, Package_QFP:LQFP-64_10x10mm_P0.5mm, symbol Video:IT6801
- removed U18: TXB0108, Package_SO:TSSOP-20_4.4x6.5mm_P0.65mm, symbol Interface:TXB0108
- removed U19: IT66121FN, Package_QFP:LQFP-64_10x10mm_P0.5mm, symbol Video:IT66121
- removed Y3, Y4: 27MHz, Crystal:Crystal_SMD_3215-2Pin_3.2x1.5mm, symbol Device:Crystal
- added C24, C25, C27, C28: 100nF, jlc_components:C0402, symbol fcBoard:C
- added C26, C29: 1uF, jlc_components:C0603, symbol fcBoard:C
- added J8, J9: HDMI, jlc_components:HDMI-SMD_HDMI-001S, symbol fcBoard:HDMI_A
- added R10, R11, R12, R13: 4.7k, jlc_components:R0402, symbol fcBoard:R
- added U8: IT6801FN, Package_QFP:LQFP-100_14x14mm_P0.5mm, symbol fcBoard:IT6801FN
- added U9: IT66121FN, Package_QFP:LQFP-100_14x14mm_P0.5mm, symbol fcBoard:IT66121FN
Connections:
- new net: C27.2, C28.1
- new net: C24.2, C25.1
- new net: C25.2, C26.1
- new net: C28.2, C29.1
- new net +5V: J9.4 (D1+)
Other:
- note added: "HDMI 1.4 Input Receiver (IT6801FN)"
- note added: "HDMI 1.4 Output Transmitter (IT66121FN)"
- title: HDMI In/Out -> HDMI Input/Output
