File: fcBoard_Peripherals.kicad_sch (KiCad schematic)
At the start: 22 parts, among them J10 MicroSD, J11 USB_Debug, J12 CAN0, J13 RS485_0, J14 CAN1, J15 RS485_1, SW1 BTN0, SW2 BTN1, U21 CP2102N, U22 SN65HVD230, U23 MAX485, U24 SN65HVD230, U25 MAX485

Commit message: 회로도 라벨
Parts:
- renumbered C13 to C38, D9 to D17, D7 to D18, D8 to D19, D10 to D20, J11 to J25, J10 to J26, J14 to J27, J13 to J28, J12 to J29, J15 to J30, R12 to R25, R14 to R26, R13 to R27, R11 to R28, SW2 to SW3, SW1 to SW4, U24 to U46, U21 to U47, U23 to U48, U25 to U49, U22 to U50
