File: fcBoard_Peripherals.kicad_sch (KiCad schematic)
At the start: 22 parts, among them J10 MicroSD, J11 USB_Debug, J12 CAN0, J13 RS485_0, J14 CAN1, J15 RS485_1, SW1 BTN0, SW2 BTN1, U21 CP2102N, U22 SN65HVD230, U23 MAX485, U24 SN65HVD230, U25 MAX485

Commit message: ㅊ
Parts:
- removed C13: 100nF, Capacitor_SMD:C_0402_1005Metric, symbol Device:C
- removed D10: LED_USER3, LED_SMD:LED_0603_1608Metric, symbol Device:LED
- removed D7: LED_USER0, LED_SMD:LED_0603_1608Metric, symbol Device:LED
- removed D8: LED_USER1, LED_SMD:LED_0603_1608Metric, symbol Device:LED
- removed D9: LED_USER2, LED_SMD:LED_0603_1608Metric, symbol Device:LED
- removed J10: MicroSD, Connector_Card:microSD_HC_Wuerth_693072010801, symbol Connector:MicroSD_Card
- removed J11: USB_Debug, Connector_PinHeader_2.54mm:PinHeader_1x02_P2.54mm_Vertical, symbol Connector:USB_B_Micro
- removed J12: CAN0, Connector_PinHeader_2.54mm:PinHeader_1x02_P2.54mm_Vertical, symbol Connector:Screw_Terminal_01x03
- removed J13: RS485_0, Connector_PinHeader_2.54mm:PinHeader_1x02_P2.54mm_Vertical, symbol Connector:Screw_Terminal_01x03
- removed J14: CAN1, Connector_PinHeader_2.54mm:PinHeader_1x02_P2.54mm_Vertical, symbol Connector:Screw_Terminal_01x03
- removed J15: RS485_1, Connector_PinHeader_2.54mm:PinHeader_1x02_P2.54mm_Vertical, symbol Connector:Screw_Terminal_01x03
- removed R11, R12, R13, R14: 470R, Resistor_SMD:R_0402_1005Metric, symbol Device:R
- removed SW1: BTN0, Button_Switch_SMD:SW_SPST_TL3342, symbol Switch:SW_Push
- removed SW2: BTN1, Button_Switch_SMD:SW_SPST_TL3342, symbol Switch:SW_Push
- removed U21: CP2102N, Package_DFN_QFN:QFN-28-1EP_5x5mm_P0.5mm_EP3.35x3.35mm, symbol Interface_USB:CP2102N
- removed U22, U24: SN65HVD230, Package_SO:SOIC-8_3.9x4.9mm_P1.27mm, symbol Interface_CAN_LIN:SN65HVD230
- removed U23, U25: MAX485, Package_SO:SOIC-8_3.9x4.9mm_P1.27mm, symbol Interface_UART:MAX485
- added D10: LED_USER3, LED_SMD:LED_0603_1608Metric, symbol LED
- added D7: LED_USER0, LED_SMD:LED_0603_1608Metric, symbol LED
- added D8: LED_USER1, LED_SMD:LED_0603_1608Metric, symbol LED
- added D9: LED_USER2, LED_SMD:LED_0603_1608Metric, symbol LED
- added J10: MicroSD, Connector_Card:microSD_HC_Wuerth_693072010801, symbol MicroSD
- added J11: USB_Debug, Connector_PinHeader_2.54mm:PinHeader_1x02_P2.54mm_Vertical, symbol PinHeader_1x02
- added J12: CAN0, Connector_PinHeader_2.54mm:PinHeader_1x02_P2.54mm_Vertical, symbol PinHeader_1x02
- added J13: RS485_0, Connector_PinHeader_2.54mm:PinHeader_1x02_P2.54mm_Vertical, symbol PinHeader_1x02
- added J14: CAN1, Connector_PinHeader_2.54mm:PinHeader_1x02_P2.54mm_Vertical, symbol PinHeader_1x02
- added J15: RS485_1, Connector_PinHeader_2.54mm:PinHeader_1x02_P2.54mm_Vertical, symbol PinHeader_1x02
- added R11, R12, R13, R14: 470R, Resistor_SMD:R_0402_1005Metric, symbol R
- added SW1: BTN0, Button_Switch_SMD:SW_SPST_TL3342, symbol SW_Push
- added SW2: BTN1, Button_Switch_SMD:SW_SPST_TL3342, symbol SW_Push
- added U21: CP2102N, Package_DFN_QFN:QFN-28-1EP_5x5mm_P0.5mm_EP3.35x3.35mm, symbol CP2102N
- added U22, U24: SN65HVD230, Package_SO:SOIC-8_3.9x4.9mm_P1.27mm, symbol SN65HVD230
- added U23, U25: MAX485, Package_SO:SOIC-8_3.9x4.9mm_P1.27mm, symbol MAX485
Other:
- company: fcBoard Project -> fcBoard
- title: Peripherals -> Peripherals - CAN, RS485, MicroSD, Debug

Commit message: 45
Parts:
- added C401, C402: 100nF, Capacitor_SMD:C_0402_1005Metric, symbol Device:C
- added R14, R15, R31, R32: 120R, Resistor_SMD:R_0402_1005Metric, symbol R
- added R20, R22, R33, R34, R36: 10k, Resistor_SMD:R_0402_1005Metric, symbol R
- renumbered D7 to D1, D8 to D2, D9 to D3, D10 to D4, J15 to J10, J10 to J11, J11 to J12, J12 to J7, J14 to J8, J13 to J9, R11 to R1, R12 to R2, R13 to R3, R14 to R4, U22 to U13, U24 to U14, U23 to U15, U25 to U16, U21 to U17
Connections:
- net CAN0_H: now also R31.1
- net CAN0_L: now also R31.2
- net RS485_1_A: now also R15.1
- net RS485_1_B: now also R15.2
- net SD_CMD: now also R22.2
- net SD_DAT0: now also R33.2
- net SD_DAT1: now also R34.2
- net SD_DAT2: now also R20.2
- net SD_DAT3: now also R36.2
- new net +3V3: R20.1, R22.1, R33.1, R34.1, R36.1
Other:
- note added: "Bus Termination Resistors 120Ω for RS485 and CAN buses"
- note added: "MicroSD Pullup Resistors 10kΩ for DAT0-3, CMD"
- moved on the sheet: D1, D2, D3, D4, J10, J11, J12, J7, J8, J9, R1, R2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
