File: fcBoard_Peripherals.kicad_sch (KiCad schematic)
At the start: 21 parts, among them J10 MicroSD, J11 USB_Debug, J12 CAN0, J13 RS485_0, J14 CAN1, J15 RS485_1, SW1 BTN0, SW2 BTN1, U21 CP2102N, U22 SN65HVD230, U23 MAX485, U24 SN65HVD230, U25 MAX485

Commit message: 45
Parts:
- removed D10: LED_USER3, LED_SMD:LED_0603_1608Metric, symbol LED
- removed D7: LED_USER0, LED_SMD:LED_0603_1608Metric, symbol LED
- removed D8: LED_USER1, LED_SMD:LED_0603_1608Metric, symbol LED
- removed D9: LED_USER2, LED_SMD:LED_0603_1608Metric, symbol LED
- removed J10: MicroSD, Connector_Card:microSD_HC_Wuerth_693072010801, symbol MicroSD
- removed J11: USB_Debug, Connector_PinHeader_2.54mm:PinHeader_1x02_P2.54mm_Vertical, symbol PinHeader_1x02
- removed J12: CAN0, Connector_PinHeader_2.54mm:PinHeader_1x02_P2.54mm_Vertical, symbol PinHeader_1x02
- removed J13: RS485_0, Connector_PinHeader_2.54mm:PinHeader_1x02_P2.54mm_Vertical, symbol PinHeader_1x02
- removed J14: CAN1, Connector_PinHeader_2.54mm:PinHeader_1x02_P2.54mm_Vertical, symbol PinHeader_1x02
- removed J15: RS485_1, Connector_PinHeader_2.54mm:PinHeader_1x02_P2.54mm_Vertical, symbol PinHeader_1x02
- removed R11, R12, R13, R14: 470R, Resistor_SMD:R_0402_1005Metric, symbol R
- removed SW1: BTN0, Button_Switch_SMD:SW_SPST_TL3342, symbol SW_Push
- removed SW2: BTN1, Button_Switch_SMD:SW_SPST_TL3342, symbol SW_Push
- removed U21: CP2102N, Package_DFN_QFN:QFN-28-1EP_5x5mm_P0.5mm_EP3.35x3.35mm, symbol CP2102N
- removed U22, U24: SN65HVD230, Package_SO:SOIC-8_3.9x4.9mm_P1.27mm, symbol SN65HVD230
- removed U23, U25: MAX485, Package_SO:SOIC-8_3.9x4.9mm_P1.27mm, symbol MAX485
- added C30: 100nF, jlc_components:C0402, symbol fcBoard:C
- added D10: YELLOW, jlc_components:LED0603-RD, symbol fcBoard:LED
- added D7: RED, jlc_components:LED0603-RD, symbol fcBoard:LED
- added D8: GREEN, jlc_components:LED0603-RD, symbol fcBoard:LED
- added D9: BLUE, jlc_components:LED0603-RD, symbol fcBoard:LED
- added J10: USB_C, jlc_components:USB-C-SMD_TYPE-C-31-M-12, symbol fcBoard:USB_C
- added J11: 2x10, jlc_components:HDR-TH_20P-P2.54-V-2X10, symbol fcBoard:Conn_2x10
- added R14, R15: 100R, jlc_components:R0402, symbol fcBoard:R
- added R16, R17, R18, R19: 330R, jlc_components:R0402, symbol fcBoard:R
- added R20, R21: 10k, jlc_components:R0402, symbol fcBoard:R
- added SW1, SW2: SW_Push, jlc_components:SW-SMD_L4.0-W4.0-P2.20, symbol fcBoard:SW_Push
- added U10, U11: MAX485ESA, Package_SO:SOIC-8_3.9x4.9mm_P1.27mm, symbol fcBoard:MAX485
- added U12: CP2102N-A02-GQFN24, Package_DFN_QFN:QFN-28-1EP_5x5mm_P0.5mm_EP3.35x3.35mm, symbol fcBoard:CP2102N
Connections:
- new net: R16.2, R17.1
- new net: R17.2, R18.1
- new net: R18.2, R19.1
Other:
- note added: "GPIO Header (2x10, 2.54mm)"
- note added: "RS485 Interface #1"
- note added: "RS485 Interface #2"
- note added: "USB to UART Bridge (Debug Console)"
- note added: "User Buttons"
- note added: "User LEDs"
- company: fcBoard -> fcBoard Project
- title: Peripherals - CAN, RS485, MicroSD, Debug -> Board Peripherals
