File: fcBoard_Power.kicad_sch (KiCad schematic)
At the start: 24 parts, among them J16 DC_12V, U26 LM2596S-ADJ, U27 LM2596S-ADJ, U28 LM2596S-5

Commit message: 45
Parts:
- removed C21, C23: 220uF, Capacitor_SMD:C_0402_1005Metric, symbol Device:CP
- removed C22: 470uF, Capacitor_SMD:C_0402_1005Metric, symbol Device:CP
- removed L5: 33uH, Inductor_SMD:L_Bourns_SRN6045TA, symbol Device:L
- removed R15: 100, Resistor_SMD:R_0402_1005Metric, symbol Device:R
- removed R20: 1.5K, Resistor_SMD:R_0402_1005Metric, symbol Device:R
- added C1, C2: 220uF, Capacitor_SMD:C_0402_1005Metric, symbol Device:CP
- added L1: 33uH, Inductor_SMD:L_Bourns_SRN6045TA, symbol Device:L
- added R5, R6, R7: 10kΩ, Resistor_SMD:R_0402_1005Metric, symbol Device:R
- added R8: 1kΩ, Resistor_SMD:R_0402_1005Metric, symbol Device:R
- added R9: 470Ω, Resistor_SMD:R_0402_1005Metric, symbol Device:R
- D11, D13, D14: footprint LED_SMD:LED_0603_1608Metric -> Diode_SMD:D_SMA
- R16: value 1.5K -> 1.2k
- R17: value 1K -> 2k
- R19: value 3.3K -> 100
Connections:
- net +1V8: now also D11.2 (A), C2.1, R9.1; no longer R17.1
- net +3V3: now also D13.2 (A), R17.1, C1.1, L1.2; no longer R19.1
- net +5V: now also U28.4 (FB)
- net GND: now also R16.1, R19.2, C1.2, C2.2, R8.1; no longer R16.2
- net at D16.2 (A): now also R19.1
- net at L4.1, U27.2 (OUT): no longer D11.2 (A)
- net +12V_IN: now reaches J16.1, U26.1 (VIN), U27.1 (VIN), U28.1 (VIN)
- net +12V_IN: now also R5.2, R6.2, R7.2
- net at U27.4 (FB): now also R8.2, R9.2; no longer R17.2
- net at U26.2 (OUT): now also L1.1; no longer D13.2 (A)
- net at U26.5 (~{ON}/OFF): now also R6.1
- net at U27.5 (~{ON}/OFF): now also R7.1
- net at U28.5 (~{ON}/OFF): now also R5.1
- new net: R16.2, R17.2, U26.4 (FB)
Other:
- moved on the sheet: C20, D11, D12, D13, D14, D15, D16, J16, L4, L6, R18, R19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
