File: fcBoard_Power.kicad_sch (KiCad schematic)
At the start: 24 parts, among them J1 DC_12V, U1 LM2596S-5, U2 LM2596S-ADJ, U3 LM2596S-ADJ

Commit message: 45
Parts:
- removed C1: 470uF, Capacitor_SMD:C_0402_1005Metric, symbol Device:CP
- removed C2, C3, C4: 220uF, Capacitor_SMD:C_0402_1005Metric, symbol Device:CP
- removed D1: LED_5V, LED_SMD:LED_0603_1608Metric, symbol Device:LED
- removed D2, D4, D6: SS34, LED_SMD:LED_0603_1608Metric, symbol Device:D_Schottky
- removed D3: LED_3V3, LED_SMD:LED_0603_1608Metric, symbol Device:LED
- removed D5: LED_1V8, LED_SMD:LED_0603_1608Metric, symbol Device:LED
- removed J1: DC_12V, Connector_BarrelJack:BarrelJack_Horizontal, symbol Connector:Barrel_Jack_Switch
- removed L1, L2, L3: 33uH, Inductor_SMD:L_Bourns_SRN6045TA, symbol Device:L
- removed R1, R5: 1K, Resistor_SMD:R_0402_1005Metric, symbol Device:R
- removed R2: 3.3K, Resistor_SMD:R_0402_1005Metric, symbol Device:R
- removed R3: 470, Resistor_SMD:R_0402_1005Metric, symbol Device:R
- removed R4, R7: 1.5K, Resistor_SMD:R_0402_1005Metric, symbol Device:R
- removed R6: 100, Resistor_SMD:R_0402_1005Metric, symbol Device:R
- removed U1: LM2596S-5, Package_TO_SOT_SMD:TO-263-5_TabPin3, symbol Regulator_Switching:LM2596S-5
- removed U2, U3: LM2596S-ADJ, Package_TO_SOT_SMD:TO-263-5_TabPin3, symbol Regulator_Switching:LM2596S-ADJ
- added C1: 470uF/25V, jlc_components:CAP-SMD_BD10.0-L10.0-W10.0-LS11.2-FD, symbol fcBoard:CP
- added C2, C3, C4: 100nF, jlc_components:C0402, symbol fcBoard:C
- added C5, C6, C7: 220uF/16V, jlc_components:CAP-SMD_BD8.0-L8.3-W8.3-LS9.0-FD, symbol fcBoard:CP
- added D1, D2, D3: SS34, jlc_components:SMA_L4.3-W2.6-LS5.2-RD, symbol fcBoard:D_Schottky
- added D4, D5: GREEN, jlc_components:LED0603-RD, symbol fcBoard:LED
- added D6: RED, jlc_components:LED0603-RD, symbol fcBoard:LED
- added J1: DC_12V, Connector_BarrelJack:BarrelJack_Horizontal, symbol fcBoard:Barrel_Jack
- added L1, L2, L3: 33uH, jlc_components:IND-SMD_L7.3-W7.3, symbol fcBoard:L
- added R1: 1.5k, jlc_components:R0402, symbol fcBoard:R
- added R2, R4: 1k, jlc_components:R0402, symbol fcBoard:R
- added R3, R6: 470R, jlc_components:R0402, symbol fcBoard:R
- added R5, R7: 330R, jlc_components:R0402, symbol fcBoard:R
- added U1: LM2596S-5.0, Package_TO_SOT_SMD:TO-263-5_TabPin3, symbol fcBoard:LM2596S-5
- added U2, U3: LM2596S-ADJ, Package_TO_SOT_SMD:TO-263-5_TabPin3, symbol fcBoard:LM2596S-ADJ
Connections:
- new net: R3.2, R4.1
- new net: R1.2, R2.1
Other:
- note added: "1.8V @ 3A Output"
- note added: "12V DC Input 5A minimum"
- note added: "3.3V @ 3A Output"
- note added: "5V @ 3A Output"
