File: fcBoard_USB.kicad_sch (KiCad schematic)
At the start: 14 parts, among them J2 USB_A, J3 USB_A, J4 USB_A, J5 USB_A, U10 TPD4S012, U11 TPS2041B, U12 TPD4S012, U13 TPS2041B, U4 TPD4S012, U5 TPS2041B, U6 USB3320, U7 USB5744, U8 TPD4S012, U9 TPS2041B

Commit message: 2121
Parts:
- removed J2, J3, J4, J5: USB_A, Connector_USB:USB_A_Stewart_SS-52100-001_Horizontal, symbol Connector:USB_A
- removed U10, U12, U4, U8: TPD4S012, Package_DFN_QFN:UQFN-10_1.4x1.8mm_P0.4mm, symbol Power_Protection:TPD4S012
- removed U11, U13, U5, U9: TPS2041B, Package_TO_SOT_SMD:SOT-23-5, symbol Power_Management:TPS2041B
- removed U6: USB3320, Package_DFN_QFN:QFN-32-1EP_5x5mm_P0.5mm_EP3.1x3.1mm, symbol Interface_USB:USB3320
- removed U7: USB5744, Package_DFN_QFN:QFN-48-1EP_6x6mm_P0.4mm_EP4.25x4.25mm, symbol Interface_USB:USB5744
- added J2, J3, J4, J5: USB_A, Connector_USB:USB_A_Stewart_SS-52100-001_Horizontal, symbol USB_A
- added U10, U12, U4, U8: TPD4S012, Package_DFN_QFN:UQFN-10_1.4x1.8mm_P0.4mm, symbol TPD4S012
- added U11, U13, U5, U9: TPS2041B, Package_TO_SOT_SMD:SOT-23-5, symbol TPS2041B
- added U6: USB3320, Package_DFN_QFN:QFN-32-1EP_5x5mm_P0.5mm_EP3.1x3.1mm, symbol USB3320
- added U7: USB5744, Package_DFN_QFN:QFN-48-1EP_6x6mm_P0.4mm_EP4.25x4.25mm, symbol USB5744
Connections:
- net +3V3: now also U10.6 (VCC), U12.6 (VCC), U4.6 (VCC), U8.6 (VCC)
- net +5V: now also U11.1 (VIN), U13.1 (VIN), U5.1 (VIN), U9.1 (VIN)
- net GND: now also J2.4 (GND), J3.4 (GND), J4.4 (GND), J5.4 (GND), U10.5 (GND), U11.5 (GND), U12.5 (GND), U13.5 (GND), U4.5 (GND), U5.5 (GND), U6.15 (GND), U7.21 (GND), U8.5 (GND), U9.5 (GND)
Other:
- company: fcBoard Project -> fcBoard
- title: USB 3.0 Hub -> USB Subsystem

Commit message: 회로도 라벨
Parts:
- renumbered J5 to J?, J3 to J?, J4 to J?, J2 to J?, U9 to U?, U10 to U?, U11 to U?, U12 to U?, U6 to U?, U13 to U?, U5 to U?, U4 to U?, U7 to U?, U8 to U?
Other:
- moved on the sheet: U?
