File: fcBoard_USB.kicad_sch (KiCad schematic)
At the start: 14 parts, among them J2 USB_A, J3 USB_A, J4 USB_A, J5 USB_A, U10 TPD4S012, U11 TPS2041B, U12 TPD4S012, U13 TPS2041B, U4 TPD4S012, U5 TPS2041B, U6 USB3320, U7 USB5744, U8 TPD4S012, U9 TPS2041B

Commit message: 45
Parts:
- added C201, C203, C205, C207, C209: 100nF, Capacitor_SMD:C_0402_1005Metric, symbol Device:C
- added C202, C204, C206, C208, C210: 10uF, Capacitor_SMD:C_0603_1608Metric, symbol Device:C
- U2: renamed from U7; footprint Package_DFN_QFN:QFN-48-1EP_6x6mm_P0.4mm_EP4.25x4.25mm -> Package_DFN_QFN:QFN-48-1EP_7x7mm_P0.5mm_EP5.6x5.6mm
- renumbered J2 to J1, J3 to J2, J4 to J3, J5 to J4, U6 to U1, U13 to U10, U4 to U3, U8 to U4, U10 to U5, U12 to U6, U5 to U7, U9 to U8, U11 to U9
Connections:
- net +5V: no longer U8.1 (VIN)
- net ULPI_CLK: now also U2.1 (CLK)
- net ULPI_D0: now also U2.5 (DATA0)
- net ULPI_D1: now also U2.6 (DATA1)
- net ULPI_D2: now also U2.7 (DATA2)
- net ULPI_D3: now also U2.8 (DATA3)
- net ULPI_D4: now also U2.9 (DATA4)
- net ULPI_D5: now also U2.10 (DATA5)
- net ULPI_D6: now also U2.11 (DATA6)
- net ULPI_D7: now also U2.12 (DATA7)
- net ULPI_DIR: now also U2.2 (DIR)
- net ULPI_NXT: now also U2.3 (NXT)
- net ULPI_STP: now also U2.4 (STP)
- net USB3_VBUS_EN: now reaches U9.3 (EN)
- net USB3_OC: now reaches U9.4 (FAULT)
- net USB1_VBUS_EN: now reaches U7.3 (EN)
- net USB1_OC: now reaches U7.4 (FAULT)
- net USB4_VBUS_EN: now reaches U10.3 (EN)
- net USB4_OC: now reaches U10.4 (FAULT)
- net USB2_VBUS_EN: now reaches U8.3 (EN)
- net USB2_OC: now reaches U8.4 (FAULT)
Other:
- note added: "USB3320 (ULPI PHY) Decoupling: C207-C210: VDD33, VDD18 100nF + 10uF per rail"
- note added: "USB5744 (USB 3.0 Hub) Decoupling: C201-C206: VDD33, VDD18, VDDA 100nF + 10uF per rail"
- moved on the sheet: J1, J2, J3, J4, U1, U10, U2, U3, U4, U5, U6, U7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
