File: fcBoard.kicad_pcb (KiCad board)
At the start: 6 copper layers, 150 x 100 mm, 4 parts

Commit message: 1
Parts:
- MH1, MH2, MH3, MH4: value MountingHole_3.2mm_M3 -> MountingHole_M3; footprint MountingHole:MountingHole_3.2mm_M3_Pad_Via -> MountingHole:MountingHole_3.2mm_M3_Pad
Other:
- net class Default removed
- net class HighSpeed removed
- net class Power removed
- board text added: "150mm x 100mm"
- board text removed: "100mm"
- board text removed: "150mm"
Changed lines of the file:
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@@
   (net 5 "+1V8")
   (net 6 "+1V2")
-  (net_class "Default" "Default net class"
-    (clearance 0.127)
-    (trace_width 0.2)
-    (via_dia 0.6)
-    (via_drill 0.3)
-    (uvia_dia 0.3)
-    (uvia_drill 0.1)
+  (gr_line
+    (start 3.0 0)
+    (end 147.0 0)
+    (layer "Edge.Cuts")
+    (stroke (width 0.1) (type solid))
   )
-  (net_class "Power" "Power distribution"
-    (clearance 0.2)
-    (trace_width 0.5)
-    (via_dia 0.8)
-    (via_drill 0.4)
-    (uvia_dia 0.3)
-    (uvia_drill 0.1)
+  (gr_line
+    (start 150.0 3.0)
+    (end 150.0 97.0)
+    (layer "Edge.Cuts")
+    (stroke (width 0.1) (type solid))
   )
-  (net_class "HighSpeed" "USB3, HDMI differential pairs"
-    (clearance 0.127)
-    (trace_width 0.15)
-    (via_dia 0.5)
-    (via_drill 0.25)
-    (uvia_dia 0.3)
-    (uvia_drill 0.1)
-    (diff_pair_width 0.15)
-    (diff_pair_gap 0.15)
+  (gr_line
+    (start 147.0 100.0)
+    (end 3.0 100.0)
+    (layer "Edge.Cuts")
+    (stroke (width 0.1) (type solid))
   )
-  ; Board Outline - 150mm x 100mm with 3mm corner radius
-  (gr_arc
-    (start 3.0 0)
-    (mid 0.8787 0.8787)
+  (gr_line
+    (start 0 97.0)
     (end 0 3.0)
     (layer "Edge.Cuts")
     (stroke (width 0.1) (type solid))
   )
-  (gr_line
-    (start 0 3.0)
-    (end 0 97.0)
+  (gr_arc
+    (start 3.0 0)
+    (mid 0.879 0.879)
+    (end 0 3.0)
+    (layer "Edge.Cuts")
+    (stroke (width 0.1) (type solid))
+  )
+  (gr_arc
+    (start 150.0 3.0)
+    (mid 149.121 0.879)
+    (end 147.0 0)
+    (layer "Edge.Cuts")
+    (stroke (width 0.1) (type solid))
+  )
+  (gr_arc
+    (start 147.0 100.0)
+    (mid 149.121 99.121)
+    (end 150.0 97.0)
     (layer "Edge.Cuts")
     (stroke (width 0.1) (type solid))
@@
   (gr_arc
     (start 0 97.0)
-    (mid 0.8787 99.1213)
+    (mid 0.879 99.121)
     (end 3.0 100.0)
     (layer "Edge.Cuts")
     (stroke (width 0.1) (type solid))
   )
-  (gr_line
-    (start 3.0 100.0)
-    (end 147.0 100.0)
-    (layer "Edge.Cuts")
-    (stroke (width 0.1) (type solid))
-  )
-  (gr_arc
-    (start 147.0 100.0)
-    (mid 149.1213 99.1213)
-    (end 150.0 97.0)
-    (layer "Edge.Cuts")
-    (stroke (width 0.1) (type solid))
-  )
-  (gr_line
-    (start 150.0 97.0)
-    (end 150.0 3.0)
-    (layer "Edge.Cuts")
-    (stroke (width 0.1) (type solid))
-  )
-  (gr_arc
-    (start 150.0 3.0)
-    (mid 149.1213 0.8787)
-    (end 147.0 0)
-    (layer "Edge.Cuts")
-    (stroke (width 0.1) (type solid))
-  )
-  (gr_line
-    (start 147.0 0)
-    (end 3.0 0)
-    (layer "Edge.Cuts")
-    (stroke (width 0.1) (type solid))
-  )
-  (footprint "MountingHole:MountingHole_3.2mm_M3_Pad_Via" (layer "F.Cu")
+  (footprint "MountingHole:MountingHole_3.2mm_M3_Pad" (layer "F.Cu")
     (at 5.0 5.0)
-    (property "Reference" "MH1" (at 0 -4) (layer "F.SilkS") (effects (font (size 1 1) (thickness 0.15))))
-    (property "Value" "MountingHole_3.2mm_M3" (at 0 4) (layer "F.Fab") (effects (font (size 1 1) (thickness 0.15))))
-    (property "Footprint" "MountingHole:MountingHole_3.2mm_M3_Pad_Via" (at 0 0 0) (unlocked yes) (layer "F.Fab") (hide yes) (effects (font (size 1 1) (thickness 0.15))))
-    (attr exclude_from_pos_files)
+    (property "Reference" "MH1" (at 0 -4 0) (layer "F.SilkS") (effects (font (size 1 1) (thickness 0.15))))
+    (property "Value" "MountingHole_M3" (at 0 4 0) (layer "F.Fab") (effects (font (size 1 1) (thickness 0.15))))
+    (property "Footprint" "MountingHole:MountingHole_3.2mm_M3_Pad" (at 0 0 0) (layer "F.Fab") (hide yes) (effects (font (size 1 1) (thickness 0.15))))
+    (attr exclude_from_pos_files exclude_from_bom)
     (fp_circle
       (center 0 0)
@@
     )
   )
-  (footprint "MountingHole:MountingHole_3.2mm_M3_Pad_Via" (layer "F.Cu")
+  (footprint "MountingHole:MountingHole_3.2mm_M3_Pad" (layer "F.Cu")
     (at 145.0 5.0)
-    (property "Reference" "MH2" (at 0 -4) (layer "F.SilkS") (effects (font (size 1 1) (thickness 0.15))))
-    (property "Value" "MountingHole_3.2mm_M3" (at 0 4) (layer "F.Fab") (effects (font (size 1 1) (thickness 0.15))))
-    (property "Footprint" "MountingHole:MountingHole_3.2mm_M3_Pad_Via" (at 0 0 0) (unlocked yes) (layer "F.Fab") (hide yes) (effects (font (size 1 1) (thickness 0.15))))
-    (attr exclude_from_pos_files)
+    (property "Reference" "MH2" (at 0 -4 0) (layer "F.SilkS") (effects (font (size 1 1) (thickness 0.15))))
+    (property "Value" "MountingHole_M3" (at 0 4 0) (layer "F.Fab") (effects (font (size 1 1) (thickness 0.15))))
+    (property "Footprint" "MountingHole:MountingHole_3.2mm_M3_Pad" (at 0 0 0) (layer "F.Fab") (hide yes) (effects (font (size 1 1) (thickness 0.15))))
+    (attr exclude_from_pos_files exclude_from_bom)
     (fp_circle
       (center 0 0)
@@
     )
   )
-  (footprint "MountingHole:MountingHole_3.2mm_M3_Pad_Via" (layer "F.Cu")
+  (footprint "MountingHole:MountingHole_3.2mm_M3_Pad" (layer "F.Cu")
     (at 5.0 95.0)
-    (property "Reference" "MH3" (at 0 -4) (layer "F.SilkS") (effects (font (size 1 1) (thickness 0.15))))
-    (property "Value" "MountingHole_3.2mm_M3" (at 0 4) (layer "F.Fab") (effects (font (size 1 1) (thickness 0.15))))
-    (property "Footprint" "MountingHole:MountingHole_3.2mm_M3_Pad_Via" (at 0 0 0) (unlocked yes) (layer "F.Fab") (hide yes) (effects (font (size 1 1) (thickness 0.15))))
-    (attr exclude_from_pos_files)
+    (property "Reference" "MH3" (at 0 -4 0) (layer "F.SilkS") (effects (font (size 1 1) (thickness 0.15))))
+    (property "Value" "MountingHole_M3" (at 0 4 0) (layer "F.Fab") (effects (font (size 1 1) (thickness 0.15))))
+    (property "Footprint" "MountingHole:MountingHole_3.2mm_M3_Pad" (at 0 0 0) (layer "F.Fab") (hide yes) (effects (font (size 1 1) (thickness 0.15))))
+    (attr exclude_from_pos_files exclude_from_bom)
     (fp_circle
       (center 0 0)
@@
     )
   )
-  (footprint "MountingHole:MountingHole_3.2mm_M3_Pad_Via" (layer "F.Cu")
+  (footprint "MountingHole:MountingHole_3.2mm_M3_Pad" (layer "F.Cu")
     (at 145.0 95.0)
-    (property "Reference" "MH4" (at 0 -4) (layer "F.SilkS") (effects (font (size 1 1) (thickness 0.15))))
-    (property "Value" "MountingHole_3.2mm_M3" (at 0 4) (layer "F.Fab") (effects (font (size 1 1) (thickness 0.15))))
-    (property "Footprint" "MountingHole:MountingHole_3.2mm_M3_Pad_Via" (at 0 0 0) (unlocked yes) (layer "F.Fab") (hide yes) (effects (font (size 1 1) (thickness 0.15))))
-    (attr exclude_from_pos_files)
+    (property "Reference" "MH4" (at 0 -4 0) (layer "F.SilkS") (effects (font (size 1 1) (thickness 0.15))))
+    (property "Value" "MountingHole_M3" (at 0 4 0) (layer "F.Fab") (effects (font (size 1 1) (thickness 0.15))))
+    (property "Footprint" "MountingHole:MountingHole_3.2mm_M3_Pad" (at 0 0 0) (layer "F.Fab") (hide yes) (effects (font (size 1 1) (thickness 0.15))))
+    (attr exclude_from_pos_files exclude_from_bom)
     (fp_circle
       (center 0 0)
@@
     )
   )
-  ; Board dimension annotations
-  (gr_text "150mm"
-    (at 75.0 105.0)
-    (layer "Dwgs.User")
-    (effects (font (size 2 2) (thickness 0.3)) (justify center))
+  (gr_text "150mm x 100mm"
+    (at 75.0 108.0 0)
+    (layer "Cmts.User")
+    (effects (font (size 2 2) (thickness 0.3)))
   )
-  (gr_text "100mm"
-    (at -5 50.0 90)
-    (layer "Dwgs.User")
-    (effects (font (size 2 2) (thickness 0.3)) (justify center))
-  )
-  ; Power plane zones (In1.Cu = GND, In2.Cu = +3V3/+5V, In4.Cu = GND)
-  ; Zones will be created after component placement
 )

Commit message: 45
Parts:
- removed MH1, MH2, MH3, MH4: MountingHole_M3, MountingHole:MountingHole_3.2mm_M3_Pad
- added C1: 220uF, Capacitor_SMD:C_0402_1005Metric, F.Cu at (211.6, 202.1)
- added C101: 20pF, Capacitor_SMD:C_0402_1005Metric, F.Cu at (285.0, 126.8)
- added C102: 20pF, Capacitor_SMD:C_0402_1005Metric, F.Cu at (285.0, 128.7)
- added C103: 20pF, Capacitor_SMD:C_0402_1005Metric, F.Cu at (285.0, 130.7)
- added C104: 20pF, Capacitor_SMD:C_0402_1005Metric, F.Cu at (285.0, 132.7)
- added C111: 100nF, Capacitor_SMD:C_0402_1005Metric, F.Cu at (285.0, 134.7)
- added C112: 10uF, Capacitor_SMD:C_0603_1608Metric, F.Cu at (281.5, 127.0)
- added C113: 100nF, Capacitor_SMD:C_0402_1005Metric, F.Cu at (287.8, 126.8)
- added C114: 10uF, Capacitor_SMD:C_0603_1608Metric, F.Cu at (281.5, 129.6)
- added C115: 100nF, Capacitor_SMD:C_0402_1005Metric, F.Cu at (287.8, 128.7)
- added C116: 10uF, Capacitor_SMD:C_0603_1608Metric, F.Cu at (281.5, 132.1)
- added C121: 100nF, Capacitor_SMD:C_0402_1005Metric, F.Cu at (287.8, 130.7)
- added C122: 10uF, Capacitor_SMD:C_0603_1608Metric, F.Cu at (281.5, 134.6)
- added C123: 100nF, Capacitor_SMD:C_0402_1005Metric, F.Cu at (287.8, 132.7)
- added C124: 10uF, Capacitor_SMD:C_0603_1608Metric, F.Cu at (281.5, 137.1)
- added C125: 100nF, Capacitor_SMD:C_0402_1005Metric, F.Cu at (287.8, 134.7)
- added C126: 10uF, Capacitor_SMD:C_0603_1608Metric, F.Cu at (281.5, 139.6)
- added C2: 220uF, Capacitor_SMD:C_0402_1005Metric, F.Cu at (187.4, 196.5)
- added C20: 220uF, Capacitor_SMD:C_0402_1005Metric, F.Cu at (226.9, 198.5)
- added C201: 100nF, Capacitor_SMD:C_0402_1005Metric, F.Cu at (299.6, 126.8)
- added C202: 10uF, Capacitor_SMD:C_0603_1608Metric, F.Cu at (296.2, 127.0)
- added C203: 100nF, Capacitor_SMD:C_0402_1005Metric, F.Cu at (299.6, 128.7)
- added C204: 10uF, Capacitor_SMD:C_0603_1608Metric, F.Cu at (296.2, 129.6)
- added C205: 100nF, Capacitor_SMD:C_0402_1005Metric, F.Cu at (299.6, 130.7)
- added C206: 10uF, Capacitor_SMD:C_0603_1608Metric, F.Cu at (296.2, 132.1)
- added C207: 100nF, Capacitor_SMD:C_0402_1005Metric, F.Cu at (299.6, 132.7)
- added C208: 10uF, Capacitor_SMD:C_0603_1608Metric, F.Cu at (296.2, 134.6)
- added C209: 100nF, Capacitor_SMD:C_0402_1005Metric, F.Cu at (299.6, 134.7)
- added C210: 10uF, Capacitor_SMD:C_0603_1608Metric, F.Cu at (296.2, 137.1)
- added C3: 10uF, Capacitor_SMD:C_0603_1608Metric, F.Cu at (112.8, 158.9)
- added C301: 100nF, Capacitor_SMD:C_0402_1005Metric, F.Cu at (285.0, 143.8)
- added C302: 10uF, Capacitor_SMD:C_0603_1608Metric, F.Cu at (281.5, 144.1)
- added C303: 100nF, Capacitor_SMD:C_0402_1005Metric, F.Cu at (285.0, 145.8)
- added C304: 10uF, Capacitor_SMD:C_0603_1608Metric, F.Cu at (281.5, 146.6)
- added C305: 100nF, Capacitor_SMD:C_0402_1005Metric, F.Cu at (285.0, 147.8)
- added C306: 10uF, Capacitor_SMD:C_0603_1608Metric, F.Cu at (281.5, 149.1)
- added C307: 100nF, Capacitor_SMD:C_0402_1005Metric, F.Cu at (285.0, 149.7)
- added C308: 10uF, Capacitor_SMD:C_0603_1608Metric, F.Cu at (281.5, 151.6)
- added C309: 100nF, Capacitor_SMD:C_0402_1005Metric, F.Cu at (285.0, 151.7)
- added C4: 100nF, Capacitor_SMD:C_0402_1005Metric, F.Cu at (119.2, 158.6)
- added C401: 100nF, Capacitor_SMD:C_0402_1005Metric, F.Cu at (292.8, 149.8)
- added C402: 100nF, Capacitor_SMD:C_0402_1005Metric, F.Cu at (292.8, 151.8)
- added D1: LED_USER0, LED_SMD:LED_0603_1608Metric, F.Cu at (349.9, 198.7)
- added D11: SS34, Diode_SMD:D_SMA, F.Cu at (190.3, 197.8)
- added D12: LED_5V, LED_SMD:LED_0603_1608Metric, F.Cu at (247.0, 197.6)
- added D13: SS34, Diode_SMD:D_SMA, F.Cu at (203.6, 197.7)
- added D14: SS34, Diode_SMD:D_SMA, F.Cu at (215.7, 197.3)
- added D15: LED_3V3, LED_SMD:LED_0603_1608Metric, F.Cu at (247.0, 201.0)
- added D16: LED_1V8, LED_SMD:LED_0603_1608Metric, F.Cu at (247.0, 204.5)
- added D2: LED_USER1, LED_SMD:LED_0603_1608Metric, F.Cu at (349.9, 192.7)
- added D3: LED_USER2, LED_SMD:LED_0603_1608Metric, F.Cu at (349.9, 186.7)
- added D4: LED_USER3, LED_SMD:LED_0603_1608Metric, F.Cu at (349.9, 180.7)
- added H1: MountingHole_3.2mm_M3, MountingHole:MountingHole_3.2mm_M3_Pad_Via, F.Cu at (156.5, 95.1)
- added H2: MountingHole_3.2mm_M3, MountingHole:MountingHole_3.2mm_M3_Pad_Via, F.Cu at (246.5, 95.1)
- added H3: MountingHole_3.2mm_M3, MountingHole:MountingHole_3.2mm_M3_Pad_Via, F.Cu at (156.5, 215.1)
- added H4: MountingHole_3.2mm_M3, MountingHole:MountingHole_3.2mm_M3_Pad_Via, F.Cu at (246.5, 215.1)
- added J1: USB_A, Connector_USB:USB_A_Stewart_SS-52100-001_Horizontal, F.Cu at (237.4, 112.2)
- added J10: RS485_1, Connector_PinHeader_2.54mm:PinHeader_1x02_P2.54mm_Vertical, F.Cu at (349.2, 225.1)
- added J101: GPIO_HEADER_1, Connector_PinHeader_2.54mm:PinHeader_2x20_P2.54mm_Vertical, F.Cu at (154.7, 103.7)
- added J102: GPIO_HEADER_1, Connector_PinHeader_2.54mm:PinHeader_2x20_P2.54mm_Vertical, F.Cu at (154.8, 158.1)
- added J103: GPIO_HEADER_1, Connector_PinHeader_2.54mm:PinHeader_2x20_P2.54mm_Vertical, F.Cu at (178.6, 97.0)
- added J11: MicroSD, Connector_Card:microSD_HC_Wuerth_693072010801, B.Cu at (316.2, 199.4)
- added J12: USB_Debug, Connector_PinHeader_2.54mm:PinHeader_1x02_P2.54mm_Vertical, F.Cu at (310.8, 216.4)
- added J15: ACU5EV_J29, fcBoard:Panasonic_AXK6A2337YG, F.Cu at (201.9, 108.1)
- added J16: DC_12V, Connector_BarrelJack:BarrelJack_Horizontal, F.Cu at (235.1, 205.5)
- added J17: ACU5EV_J30, fcBoard:Panasonic_AXK6A2337YG, F.Cu at (228.1, 145.4)
- added J18: ACU5EV_J31, fcBoard:Panasonic_AXK6A2337YG, F.Cu at (175.6, 145.4)
- added J19: ACU5EV_J32, fcBoard:Panasonic_AXK6A2337YG, F.Cu at (201.9, 182.6)
- added J2: USB_A, Connector_USB:USB_A_Stewart_SS-52100-001_Horizontal, F.Cu at (237.5, 130.0)
- added J23: HDMI_OUT, fcBoard_Connectors:HDMI_A_Contact_Technology_HDMI-19APL2_Horizontal, F.Cu at (12.3, -77.8)
- added J24: HDMI_IN, fcBoard_Connectors:HDMI_A_Contact_Technology_HDMI-19APL2_Horizontal, F.Cu at (39.8, -98.3)
- added J3: USB_A, Connector_USB:USB_A_Stewart_SS-52100-001_Horizontal, F.Cu at (237.6, 147.9)
- added J4: USB_A, Connector_USB:USB_A_Stewart_SS-52100-001_Horizontal, F.Cu at (237.6, 166.3)
- added J5: RJ45_MagJack, Connector_RJ:RJ45_Hanrun_HR911105A_Horizontal, F.Cu at (97.8, 264.7)
- added J7: CAN0, Connector_PinHeader_2.54mm:PinHeader_1x02_P2.54mm_Vertical, F.Cu at (318.2, 224.3)
- added J8: CAN1, Connector_PinHeader_2.54mm:PinHeader_1x02_P2.54mm_Vertical, F.Cu at (328.5, 224.6)
- added J9: RS485_0, Connector_PinHeader_2.54mm:PinHeader_1x02_P2.54mm_Vertical, F.Cu at (337.9, 224.9)
- added L1: 33uH, Inductor_SMD:L_Bourns_SRN6045TA, F.Cu at (209.1, 197.7)
- added L4: 33uH, Inductor_SMD:L_Bourns_SRN6045TA, F.Cu at (197.4, 197.8)
- added L6: 33uH, Inductor_SMD:L_Bourns_SRN6045TA, F.Cu at (221.3, 197.5)
- added R1: 470R, Resistor_SMD:R_0402_1005Metric, F.Cu at (356.6, 196.2)
- added R10: 10k, Resistor_SMD:R_0402_1005Metric, F.Cu at (116.3, 158.6)
- added R11: 10k, Resistor_SMD:R_0402_1005Metric, F.Cu at (116.3, 160.6)
- added R12: 10k, Resistor_SMD:R_0402_1005Metric, F.Cu at (287.9, 143.8)
- added R13: 10k, Resistor_SMD:R_0402_1005Metric, F.Cu at (287.9, 145.8)
- added R14: 120R, Resistor_SMD:R_0402_1005Metric, F.Cu at (292.8, 143.8)
- added R15: 120R, Resistor_SMD:R_0402_1005Metric, F.Cu at (292.8, 145.8)
- added R16: 1.2k, Resistor_SMD:R_0402_1005Metric, F.Cu at (209.5, 202.1)
- added R17: 2k, Resistor_SMD:R_0402_1005Metric, F.Cu at (207.2, 202.2)
- added R18: 470, Resistor_SMD:R_0402_1005Metric, F.Cu at (245.5, 201.0)
- added R19: 100, Resistor_SMD:R_0402_1005Metric, F.Cu at (245.4, 204.3)
- added R2: 470R, Resistor_SMD:R_0402_1005Metric, F.Cu at (356.6, 191.2)
- added R20: 10k, Resistor_SMD:R_0402_1005Metric, F.Cu at (292.8, 147.8)
- added R21: 1K, Resistor_SMD:R_0402_1005Metric, F.Cu at (245.3, 197.5)
- added R22: 10k, Resistor_SMD:R_0402_1005Metric, F.Cu at (295.7, 143.8)
- added R23: 4.7k, Resistor_SMD:R_0402_1005Metric, F.Cu at (290.7, 126.8)
- added R24: 4.7k, Resistor_SMD:R_0402_1005Metric, F.Cu at (290.7, 128.8)
- added R25: 10k, Resistor_SMD:R_0402_1005Metric, F.Cu at (287.9, 147.8)
- added R26: 10k, Resistor_SMD:R_0402_1005Metric, F.Cu at (290.7, 130.8)
- added R27: 27k, Resistor_SMD:R_0402_1005Metric, F.Cu at (290.7, 132.8)
- added R3: 470R, Resistor_SMD:R_0402_1005Metric, F.Cu at (356.6, 186.2)
- added R31: 120R, Resistor_SMD:R_0402_1005Metric, F.Cu at (295.7, 145.8)
- added R32: 120R, Resistor_SMD:R_0402_1005Metric, F.Cu at (295.7, 147.8)
- added R33: 10k, Resistor_SMD:R_0402_1005Metric, F.Cu at (298.6, 143.8)
- added R34: 10k, Resistor_SMD:R_0402_1005Metric, F.Cu at (298.6, 145.8)
- added R36: 10k, Resistor_SMD:R_0402_1005Metric, F.Cu at (298.6, 147.8)
- added R4: 470R, Resistor_SMD:R_0402_1005Metric, F.Cu at (356.6, 181.2)
- added R5: 10kΩ, Resistor_SMD:R_0402_1005Metric, F.Cu at (226.1, 201.9)
- added R6: 10kΩ, Resistor_SMD:R_0402_1005Metric, F.Cu at (205.0, 202.1)
- added R7: 10kΩ, Resistor_SMD:R_0402_1005Metric, F.Cu at (190.1, 202.2)
- added R8: 1kΩ, Resistor_SMD:R_0402_1005Metric, F.Cu at (194.4, 202.3)
- added R9: 470Ω, Resistor_SMD:R_0402_1005Metric, F.Cu at (192.4, 202.4)
- added SW1: BTN0, Button_Switch_SMD:SW_SPST_TL3342, F.Cu at (288.6, 218.6)
- added SW2: BTN1, Button_Switch_SMD:SW_SPST_TL3342, F.Cu at (300.4, 217.9)
- added SW3: RESET, Button_Switch_SMD:SW_Push_1TS009xxxx-xxxx-xxxx_6x6x5mm, F.Cu at (115.6, 153.8)
- added U1: USB3320, Package_DFN_QFN:QFN-32-1EP_5x5mm_P0.5mm_EP3.1x3.1mm, F.Cu at (411.6, 92.6)
- added U10: TPS2041B, Package_TO_SOT_SMD:SOT-23-5, F.Cu at (472.5, 127.1)
- added U11: RTL8211F-CG, Package_DFN_QFN:QFN-48-1EP_7x7mm_P0.5mm_EP5.6x5.6mm, F.Cu at (87.0, 259.3)
- added U12: RTL8211F-CG, Package_DFN_QFN:QFN-48-1EP_7x7mm_P0.5mm_EP5.6x5.6mm, F.Cu at (87.0, 278.0)
- added U13: SN65HVD230, Package_SO:SOIC-8_3.9x4.9mm_P1.27mm, F.Cu at (350.0, 216.8)
- added U14: SN65HVD230, Package_SO:SOIC-8_3.9x4.9mm_P1.27mm, F.Cu at (339.5, 216.7)
- added U15: MAX485, Package_SO:SOIC-8_3.9x4.9mm_P1.27mm, F.Cu at (329.1, 217.3)
- added U16: MAX485, Package_SO:SOIC-8_3.9x4.9mm_P1.27mm, F.Cu at (319.2, 217.1)
- added U17: CP2102N, Package_DFN_QFN:QFN-28-1EP_5x5mm_P0.5mm_EP3.35x3.35mm, F.Cu at (310.9, 229.3)
- added U2: USB5744, Package_DFN_QFN:QFN-48-1EP_7x7mm_P0.5mm_EP5.6x5.6mm, F.Cu at (415.0, 107.6)
- added U26: LM2596S-ADJ, Package_TO_SOT_SMD:TO-263-5_TabPin3, F.Cu at (208.0, 213.2)
- added U27: LM2596S-ADJ, Package_TO_SOT_SMD:TO-263-5_TabPin3, F.Cu at (194.4, 213.2)
- added U28: LM2596S-5, Package_TO_SOT_SMD:TO-263-5_TabPin3, F.Cu at (221.7, 213.2)
- added U3: TPD4S012, Package_DFN_QFN:UQFN-10_1.4x1.8mm_P0.4mm, F.Cu at (474.4, 65.4)
- added U4: TPD4S012, Package_DFN_QFN:UQFN-10_1.4x1.8mm_P0.4mm, F.Cu at (473.2, 96.5)
- added U41: IT66121FN, Package_QFP:LQFP-64_10x10mm_P0.5mm, F.Cu at (28.4, -42.4)
- added U42: TXB0108, Package_SO:TSSOP-20_4.4x6.5mm_P0.65mm, F.Cu at (67.5, -54.5)
- added U43: IT6801FN, Package_QFP:LQFP-64_10x10mm_P0.5mm, F.Cu at (80.9, -57.5)
- added U44: TPD12S016, Package_DFN_QFN:QFN-24-1EP_4x4mm_P0.5mm_EP2.7x2.7mm, F.Cu at (58.4, -56.3)
- added U45: TPD12S016, Package_DFN_QFN:QFN-24-1EP_4x4mm_P0.5mm_EP2.7x2.7mm, F.Cu at (38.5, -60.4)
- added U5: TPD4S012, Package_DFN_QFN:UQFN-10_1.4x1.8mm_P0.4mm, F.Cu at (472.9, 116.3)
- added U6: TPD4S012, Package_DFN_QFN:UQFN-10_1.4x1.8mm_P0.4mm, F.Cu at (466.8, 125.6)
- added U7: TPS2041B, Package_TO_SOT_SMD:SOT-23-5, F.Cu at (473.2, 71.1)
- added U8: TPS2041B, Package_TO_SOT_SMD:SOT-23-5, F.Cu at (472.9, 90.6)
- added U9: TPS2041B, Package_TO_SOT_SMD:SOT-23-5, F.Cu at (472.6, 109.2)
- added Y10: 27MHz, Crystal:Crystal_SMD_3215-2Pin_3.2x1.5mm, F.Cu at (70.8, -63.8)
- added Y9: 27MHz, Crystal:Crystal_SMD_3215-2Pin_3.2x1.5mm, F.Cu at (10.6, -46.8)
Routing:
- added copper zone on In2.Cu, net +3V3
- added copper zone on In3.Cu, net +5V
- added copper zone on B.Cu, net GND
- added copper zone on F.Cu, net GND
- added copper zone on In1.Cu, net GND
Other:
- board size 150 x 100 mm -> 100 x 130 mm
- board text added: "100mm x 130mm"
- board text removed: "150mm x 100mm"
