File: fcBoard.kicad_pcb (KiCad board)
At the start: 6 copper layers, 0 parts

Commit message: 자동화
Parts:
- added C18: 1uF, jlc_components:C0603, F.Cu at (120.0, 150.3)
- added C21: 1uF, jlc_components:C0603, F.Cu at (120.0, 153.0)
- added C26: 1uF, jlc_components:C0603, F.Cu at (128.9, 119.9)
- added C29: 1uF, jlc_components:C0603, F.Cu at (128.9, 122.6)
- added D10: YELLOW, jlc_components:LED0603-RD, F.Cu at (85.2, 158.3)
- added D4: GREEN, jlc_components:LED0603-RD, F.Cu at (94.4, 123.9)
- added D5: GREEN, jlc_components:LED0603-RD, F.Cu at (94.4, 126.6)
- added D6: RED, jlc_components:LED0603-RD, F.Cu at (94.4, 129.2)
- added D7: RED, jlc_components:LED0603-RD, F.Cu at (85.2, 150.3)
- added D8: GREEN, jlc_components:LED0603-RD, F.Cu at (85.2, 153.0)
- added D9: BLUE, jlc_components:LED0603-RD, F.Cu at (85.2, 155.6)
- added J1: DC_12V, Connector_BarrelJack:BarrelJack_Horizontal, F.Cu at (103.8, 115.3)
- added R1: 1.5k, jlc_components:R0402, F.Cu at (90.8, 123.7)
- added R10: 4.7k, jlc_components:R0402, F.Cu at (128.4, 111.0)
- added R11: 4.7k, jlc_components:R0402, F.Cu at (128.4, 113.2)
- added R12: 4.7k, jlc_components:R0402, F.Cu at (128.4, 115.3)
- added R13: 4.7k, jlc_components:R0402, F.Cu at (128.4, 117.5)
- added R14: 100R, jlc_components:R0402, F.Cu at (73.1, 150.1)
- added R15: 100R, jlc_components:R0402, F.Cu at (73.1, 152.2)
- added R16: 330R, jlc_components:R0402, F.Cu at (73.1, 154.4)
- added R17: 330R, jlc_components:R0402, F.Cu at (73.1, 156.5)
- added R18: 330R, jlc_components:R0402, F.Cu at (73.1, 158.7)
- added R19: 330R, jlc_components:R0402, F.Cu at (73.1, 160.8)
- added R2: 1k, jlc_components:R0402, F.Cu at (90.8, 125.8)
- added R20: 10k, jlc_components:R0402, F.Cu at (73.1, 163.0)
- added R21: 10k, jlc_components:R0402, F.Cu at (73.1, 165.1)
- added R3: 470R, jlc_components:R0402, F.Cu at (90.8, 128.0)
- added R4: 1k, jlc_components:R0402, F.Cu at (90.8, 130.1)
- added R5: 330R, jlc_components:R0402, F.Cu at (90.8, 132.3)
- added R6: 470R, jlc_components:R0402, F.Cu at (90.8, 134.4)
- added R7: 330R, jlc_components:R0402, F.Cu at (90.8, 136.6)
- added R8: 10k, jlc_components:R0402, F.Cu at (119.5, 155.4)
- added R9: 10k, jlc_components:R0402, F.Cu at (119.5, 157.6)
- added U1: LM2596S-5.0, Package_TO_SOT_SMD:TO-263-5_TabPin3, F.Cu at (82.3, 116.1)
- added U10: MAX485ESA, Package_SO:SOIC-8_3.9x4.9mm_P1.27mm, F.Cu at (78.9, 152.4)
- added U11: MAX485ESA, Package_SO:SOIC-8_3.9x4.9mm_P1.27mm, F.Cu at (78.9, 159.0)
- added U12: CP2102N-A02-GQFN24, Package_DFN_QFN:QFN-28-1EP_5x5mm_P0.5mm_EP3.35x3.35mm, F.Cu at (87.1, 163.2)
- added U2: LM2596S-ADJ, Package_TO_SOT_SMD:TO-263-5_TabPin3, F.Cu at (82.3, 128.5)
- added U3: LM2596S-ADJ, Package_TO_SOT_SMD:TO-263-5_TabPin3, F.Cu at (82.3, 140.8)
- added U4: USB5744, Package_DFN_QFN:QFN-56-1EP_7x7mm_P0.4mm_EP5.6x5.6mm, F.Cu at (97.8, 153.7)
- added U5: USB3320C-EZK, Package_DFN_QFN:QFN-32-1EP_5x5mm_P0.5mm_EP3.6x3.6mm, F.Cu at (96.7, 161.9)
- added U6: RTL8211F-CG, Package_DFN_QFN:QFN-48-1EP_7x7mm_P0.5mm_EP5.3x5.3mm, F.Cu at (113.4, 153.6)
- added U7: RTL8211F-CG, Package_DFN_QFN:QFN-48-1EP_7x7mm_P0.5mm_EP5.3x5.3mm, F.Cu at (113.4, 162.9)
- added U8: IT6801FN, Package_QFP:LQFP-100_14x14mm_P0.5mm, F.Cu at (117.6, 119.2)
- added U9: IT66121FN, Package_QFP:LQFP-100_14x14mm_P0.5mm, F.Cu at (117.6, 137.7)

Commit message: 자동화2
Parts:
- removed C18, C21, C26, C29: 1uF, jlc_components:C0603
- removed D10: YELLOW, jlc_components:LED0603-RD
- removed D4, D5, D8: GREEN, jlc_components:LED0603-RD
- removed D6, D7: RED, jlc_components:LED0603-RD
- removed D9: BLUE, jlc_components:LED0603-RD
- removed J1: DC_12V, Connector_BarrelJack:BarrelJack_Horizontal
- removed R1: 1.5k, jlc_components:R0402
- removed R10, R11, R12, R13: 4.7k, jlc_components:R0402
- removed R14, R15: 100R, jlc_components:R0402
- removed R16, R17, R18, R19, R5, R7: 330R, jlc_components:R0402
- removed R2, R4: 1k, jlc_components:R0402
- removed R20, R21, R8, R9: 10k, jlc_components:R0402
- removed R3, R6: 470R, jlc_components:R0402
- removed U1: LM2596S-5.0, Package_TO_SOT_SMD:TO-263-5_TabPin3
- removed U10, U11: MAX485ESA, Package_SO:SOIC-8_3.9x4.9mm_P1.27mm
- removed U12: CP2102N-A02-GQFN24, Package_DFN_QFN:QFN-28-1EP_5x5mm_P0.5mm_EP3.35x3.35mm
- removed U2, U3: LM2596S-ADJ, Package_TO_SOT_SMD:TO-263-5_TabPin3
- removed U4: USB5744, Package_DFN_QFN:QFN-56-1EP_7x7mm_P0.4mm_EP5.6x5.6mm
- removed U5: USB3320C-EZK, Package_DFN_QFN:QFN-32-1EP_5x5mm_P0.5mm_EP3.6x3.6mm
- removed U6, U7: RTL8211F-CG, Package_DFN_QFN:QFN-48-1EP_7x7mm_P0.5mm_EP5.3x5.3mm
- removed U8: IT6801FN, Package_QFP:LQFP-100_14x14mm_P0.5mm
- removed U9: IT66121FN, Package_QFP:LQFP-100_14x14mm_P0.5mm
