File: fcBoard.kicad_sch (KiCad schematic)
At the start: 0 parts

Commit message: 45
Other:
- sheet Power Supply ports: added none; removed +12V, +1V8, +3V3, +5V, GND
- note added: "ACU5EV SoM Carrier Board - Main Sheet Hierarchical Design: 1. Power Supply (12V/5V/3.3V/1.8V) 2. USB 3.0 Hub (4 ports) 3. Gigabit Ethernet (2 ports) 4. HDMI In/Out 5. Peripherals (RS485, UART, GPIO)"
- note added: "All sub-schematics use EMBEDDED symbols. No external library dependencies required. JLCPCB LCSC Part numbers included for BOM."
- note removed: "ACU5EV SoM Carrier Board - Main Sheet Hierarchical Design: 1. Power Supply 2. SoM Connectors (J29-J32) 3. USB 3.0 Hub (4 ports) 4. Gigabit Ethernet (2 ports) 5. HDMI In/Out 6. Peripherals"
- note removed: "Power Distribution: +12V to J32 (pins 107-120) +1V8 to J32 VCCO_65/66 GND to All connectors"
- note removed: "SoM Connectors (ACU5EV) J29: BANK65/66 (HDMI, MIPI, ETH PL) J30: MGT505/BANK25/26 (PCIe, SFP) J31: BANK24/44 (RS485, GPIO) J32: PS MIO/Power (USB, ETH PS, SD)"
Changed lines of the file:
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@@
 	(title_block
 		(title "ACU5EV SoM Carrier Board")
-		(date "2024-11-30")
-		(rev "0.1")
+		(date "2024-12-12")
+		(rev "1.0")
 		(company "fcBoard Project")
 		(comment 1 "Full-featured carrier board for ALINX ACU5EV SoM")
-		(comment 2 "Zynq UltraScale+ MPSoC XCZU5EV")
+		(comment 2 "Zynq UltraScale+ MPSoC XCZU5EV - Embedded Symbols")
 	)
-	(text "ACU5EV SoM Carrier Board - Main Sheet\n\nHierarchical Design:\n1. Power Supply\n2. SoM Connectors (J29-J32)\n3. USB 3.0 Hub (4 ports)\n4. Gigabit Ethernet (2 ports)\n5. HDMI In/Out\n6. Peripherals"
+	(text "All sub-schematics use EMBEDDED symbols.\nNo external library dependencies required.\nJLCPCB LCSC Part numbers included for BOM."
+		(exclude_from_sim no)
+		(at 152.4 30.48 0)
+		(effects
+			(font
+				(size 1.5 1.5)
+			)
+			(justify left)
+		)
+	)
+	(text "ACU5EV SoM Carrier Board - Main Sheet\n\nHierarchical Design:\n1. Power Supply (12V/5V/3.3V/1.8V)\n2. USB 3.0 Hub (4 ports)\n3. Gigabit Ethernet (2 ports)\n4. HDMI In/Out\n5. Peripherals (RS485, UART, GPIO)"
 		(exclude_from_sim no)
 		(at 25.4 30.48 0)
@@
 		)
 	)
-	(text "SoM Connectors (ACU5EV)\n\nJ29: BANK65/66 (HDMI, MIPI, ETH PL)\nJ30: MGT505/BANK25/26 (PCIe, SFP)\nJ31: BANK24/44 (RS485, GPIO)\nJ32: PS MIO/Power (USB, ETH PS, SD)"
+	(sheet
+		(at 152.4 76.2)
+		(size 50.8 30.48)
 		(exclude_from_sim no)
-		(at 152.4 91.44 0)
-		(effects
-			(font
-				(size 1.27 1.27)
+		(in_bom yes)
+		(on_board yes)
+		(dnp no)
+		(fields_autoplaced yes)
+		(stroke
+			(width 0.1524)
+			(type solid)
+		)
+		(fill
+			(color 194 194 255 1.0000)
+		)
+		(property "Sheetname" "Gigabit Ethernet"
+			(at 152.4 75.4884 0)
+			(effects
+				(font
+					(size 1.27 1.27)
+				)
+				(justify left bottom)
 			)
-			(justify left)
+		)
+		(property "Sheetfile" "fcBoard_Ethernet.kicad_sch"
+			(at 152.4 107.2216 0)
+			(effects
+				(font
+					(size 1.27 1.27)
+				)
+				(justify left top)
+			)
 		)
 	)
-	(text "Power Distribution:\n+12V to J32 (pins 107-120)\n+1V8 to J32 VCCO_65/66\nGND to All connectors"
+	(sheet
+		(at 215.9 76.2)
+		(size 50.8 30.48)
 		(exclude_from_sim no)
-		(at 101.6 111.76 0)
-		(effects
-			(font
-				(size 1 1)
+		(in_bom yes)
+		(on_board yes)
+		(dnp no)
+		(fields_autoplaced yes)
+		(stroke
+			(width 0.1524)
+			(type solid)
+		)
+		(fill
+			(color 255 194 194 1.0000)
+		)
+		(property "Sheetname" "HDMI In/Out"
+			(at 215.9 75.4884 0)
+			(effects
+				(font
+					(size 1.27 1.27)
+				)
+				(justify left bottom)
 			)
-			(justify left)
+		)
+		(property "Sheetfile" "fcBoard_HDMI.kicad_sch"
+			(at 215.9 107.2216 0)
+			(effects
+				(font
+					(size 1.27 1.27)
+				)
+				(justify left top)
+			)
 		)
 	)
@@
 			)
 		)
-		(pin "+12V" input
-			(at 76.2 81.28 0)
+	)
+	(sheet
+		(at 279.4 76.2)
+		(size 50.8 30.48)
+		(exclude_from_sim no)
+		(in_bom yes)
+		(on_board yes)
+		(dnp no)
+		(fields_autoplaced yes)
+		(stroke
+			(width 0.1524)
+			(type solid)
+		)
+		(fill
+			(color 255 255 255 1.0000)
+		)
+		(property "Sheetname" "Peripherals"
+			(at 279.4 75.4884 0)
 			(effects
 				(font
 					(size 1.27 1.27)
 				)
-				(justify left)
+				(justify left bottom)
 			)
 		)
-		(pin "+5V" output
-			(at 76.2 86.36 0)
+		(property "Sheetfile" "fcBoard_Peripherals.kicad_sch"
+			(at 279.4 107.2216 0)
 			(effects
 				(font
 					(size 1.27 1.27)
 				)
-				(justify left)
-			)
-		)
-		(pin "+3V3" output
-			(at 76.2 91.44 0)
-			(effects
-				(font
-					(size 1.27 1.27)
-				)
-				(justify left)
-			)
-		)
-		(pin "+1V8" output
-			(at 76.2 96.52 0)
-			(effects
-				(font
-					(size 1.27 1.27)
-				)
-				(justify left)
-			)
-		)
-		(pin "GND" passive
-			(at 76.2 101.6 0)
-			(effects
-				(font
-					(size 1.27 1.27)
-				)
-				(justify left)
-			)
-		)
-		(instances
-			(project "fcBoard"
-				(path "/e63e39d7-6ac0-4ffd-8aa3-1841a4541b55"
-					(page "2")
-				)
+				(justify left top)
 			)
 		)
 	)
 	(sheet
-		(at 25.4 119.38)
-		(size 50.8 25.4)
+		(at 88.9 76.2)
+		(size 50.8 30.48)
 		(exclude_from_sim no)
 		(in_bom yes)
@@
 		)
 		(property "Sheetname" "USB 3.0 Hub"
-			(at 25.4 118.6684 0)
+			(at 88.9 75.4884 0)
 			(effects
 				(font
@@
 		)
 		(property "Sheetfile" "fcBoard_USB.kicad_sch"
-			(at 25.4 145.3216 0)
+			(at 88.9 107.2216 0)
 			(effects
 				(font
@@
 			)
 		)
-		(instances
-			(project "fcBoard"
-				(path "/e63e39d7-6ac0-4ffd-8aa3-1841a4541b55"
-					(page "3")
-				)
-			)
-		)
-	)
-	(sheet
-		(at 25.4 154.94)
-		(size 50.8 25.4)
-		(exclude_from_sim no)
-		(in_bom yes)
-		(on_board yes)
-		(dnp no)
-		(fields_autoplaced yes)
-		(stroke
-			(width 0.1524)
-			(type solid)
-		)
-		(fill
-			(color 194 224 255 1.0000)
-		)
-		(property "Sheetname" "Gigabit Ethernet"
-			(at 25.4 154.2284 0)
-			(effects
-				(font
-					(size 1.27 1.27)
-				)
-				(justify left bottom)
-			)
-		)
-		(property "Sheetfile" "fcBoard_Ethernet.kicad_sch"
-			(at 25.4 180.8816 0)
-			(effects
-				(font
-					(size 1.27 1.27)
-				)
-				(justify left top)
-			)
-		)
-		(instances
-			(project "fcBoard"
-				(path "/e63e39d7-6ac0-4ffd-8aa3-1841a4541b55"
-					(page "4")
-				)
-			)
-		)
-	)
-	(sheet
-		(at 25.4 190.5)
-		(size 50.8 25.4)
-		(exclude_from_sim no)
-		(in_bom yes)
-		(on_board yes)
-		(dnp no)
-		(fields_autoplaced yes)
-		(stroke
-			(width 0.1524)
-			(type solid)
-		)
-		(fill
-			(color 255 194 224 1.0000)
-		)
-		(property "Sheetname" "HDMI In/Out"
-			(at 25.4 189.7884 0)
-			(effects
-				(font
-					(size 1.27 1.27)
-				)
-				(justify left bottom)
-			)
-		)
-		(property "Sheetfile" "fcBoard_HDMI.kicad_sch"
-			(at 25.4 216.4416 0)
-			(effects
-				(font
-					(size 1.27 1.27)
-				)
-				(justify left top)
-			)
-		)
-		(instances
-			(project "fcBoard"
-				(path "/e63e39d7-6ac0-4ffd-8aa3-1841a4541b55"
-					(page "5")
-				)
-			)
-		)
-	)
-	(sheet
-		(at 25.4 226.06)
-		(size 50.8 25.4)
-		(exclude_from_sim no)
-		(in_bom yes)
-		(on_board yes)
-		(dnp no)
-		(fields_autoplaced yes)
-		(stroke
-			(width 0.1524)
-			(type solid)
-		)
-		(fill
-			(color 224 194 255 1.0000)
-		)
-		(property "Sheetname" "Peripherals"
-			(at 25.4 225.3484 0)
-			(effects
-				(font
-					(size 1.27 1.27)
-				)
-				(justify left bottom)
-			)
-		)
-		(property "Sheetfile" "fcBoard_Peripherals.kicad_sch"
-			(at 25.4 252.0016 0)
-			(effects
-				(font
-					(size 1.27 1.27)
-				)
-				(justify left top)
-			)
-		)
-		(instances
-			(project "fcBoard"
-				(path "/e63e39d7-6ac0-4ffd-8aa3-1841a4541b55"
-					(page "6")
-				)
-			)
-		)

Commit message: 자동화2
Other:
- sheet Power Supply ports: added +12V, +1V8, +3V3, +5V, GND; removed none
- note added: "Power Distribution: +12V Input (DC Jack) +5V @ 3A (LM2596S-5.0) +3V3 @ 3A (LM2596S-ADJ) +1V8 @ 3A (LM2596S-ADJ)"
- note added: "SoM Connectors (ACU5EV) J29: BANK65/66 (HDMI, MIPI, ETH PL) J30: MGT505/BANK25/26 (PCIe, SFP) J31: BANK24/44 (RS485, GPIO) J32: PS MIO/Power (USB, ETH PS, SD)"
Changed lines of the file:
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@@
 	(title_block
 		(title "ACU5EV SoM Carrier Board")
-		(date "2024-12-12")
+		(date "2024-12-11")
 		(rev "1.0")
 		(company "fcBoard Project")
@@
 		(comment 2 "Zynq UltraScale+ MPSoC XCZU5EV - Embedded Symbols")
 	)
+	(text "ACU5EV SoM Carrier Board - Main Sheet\n\nHierarchical Design:\n1. Power Supply (12V/5V/3.3V/1.8V)\n2. USB 3.0 Hub (4 ports)\n3. Gigabit Ethernet (2 ports)\n4. HDMI In/Out\n5. Peripherals (RS485, UART, GPIO)"
+		(exclude_from_sim no)
+		(at 25.4 30.48 0)
+		(effects
+			(font
+				(size 2 2)
+			)
+			(justify left)
+		)
+	)
 	(text "All sub-schematics use EMBEDDED symbols.\nNo external library dependencies required.\nJLCPCB LCSC Part numbers included for BOM."
 		(exclude_from_sim no)
@@
 		)
 	)
-	(text "ACU5EV SoM Carrier Board - Main Sheet\n\nHierarchical Design:\n1. Power Supply (12V/5V/3.3V/1.8V)\n2. USB 3.0 Hub (4 ports)\n3. Gigabit Ethernet (2 ports)\n4. HDMI In/Out\n5. Peripherals (RS485, UART, GPIO)"
-		(exclude_from_sim no)
-		(at 25.4 30.48 0)
-		(effects
-			(font
-				(size 2 2)
-			)
-			(justify left)
-		)
-	)
-	(sheet
-		(at 152.4 76.2)
-		(size 50.8 30.48)
-		(exclude_from_sim no)
-		(in_bom yes)
-		(on_board yes)
-		(dnp no)
-		(fields_autoplaced yes)
-		(stroke
-			(width 0.1524)
-			(type solid)
-		)
-		(fill
-			(color 194 194 255 1.0000)
-		)
-		(property "Sheetname" "Gigabit Ethernet"
-			(at 152.4 75.4884 0)
-			(effects
-				(font
-					(size 1.27 1.27)
-				)
-				(justify left bottom)
-			)
-		)
-		(property "Sheetfile" "fcBoard_Ethernet.kicad_sch"
-			(at 152.4 107.2216 0)
-			(effects
-				(font
-					(size 1.27 1.27)
-				)
-				(justify left top)
-			)
-		)
-	)
-	(sheet
-		(at 215.9 76.2)
-		(size 50.8 30.48)
-		(exclude_from_sim no)
-		(in_bom yes)
-		(on_board yes)
-		(dnp no)
-		(fields_autoplaced yes)
-		(stroke
-			(width 0.1524)
-			(type solid)
-		)
-		(fill
-			(color 255 194 194 1.0000)
-		)
-		(property "Sheetname" "HDMI In/Out"
-			(at 215.9 75.4884 0)
-			(effects
-				(font
-					(size 1.27 1.27)
-				)
-				(justify left bottom)
-			)
-		)
-		(property "Sheetfile" "fcBoard_HDMI.kicad_sch"
-			(at 215.9 107.2216 0)
-			(effects
-				(font
-					(size 1.27 1.27)
-				)
-				(justify left top)
-			)
+	(text "SoM Connectors (ACU5EV)\n\nJ29: BANK65/66 (HDMI, MIPI, ETH PL)\nJ30: MGT505/BANK25/26 (PCIe, SFP)\nJ31: BANK24/44 (RS485, GPIO)\nJ32: PS MIO/Power (USB, ETH PS, SD)"
+		(exclude_from_sim no)
+		(at 152.4 91.44 0)
+		(effects
+			(font
+				(size 1.27 1.27)
+			)
+			(justify left)
+		)
+	)
+	(text "Power Distribution:\n+12V Input (DC Jack)\n+5V @ 3A (LM2596S-5.0)\n+3V3 @ 3A (LM2596S-ADJ)\n+1V8 @ 3A (LM2596S-ADJ)"
+		(exclude_from_sim no)
+		(at 101.6 111.76 0)
+		(effects
+			(font
+				(size 1 1)
+			)
+			(justify left)
 		)
 	)
@@
 			)
 		)
-	)
-	(sheet
-		(at 279.4 76.2)
-		(size 50.8 30.48)
-		(exclude_from_sim no)
-		(in_bom yes)
-		(on_board yes)
-		(dnp no)
-		(fields_autoplaced yes)
-		(stroke
-			(width 0.1524)
-			(type solid)
-		)
-		(fill
-			(color 255 255 255 1.0000)
+		(pin "+12V" input
+			(at 76.2 81.28 0)
+			(effects
+				(font
+					(size 1.27 1.27)
+				)
+				(justify left)
+			)
+		)
+		(pin "+5V" output
+			(at 76.2 86.36 0)
+			(effects
+				(font
+					(size 1.27 1.27)
+				)
+				(justify left)
+			)
+		)
+		(pin "+3V3" output
+			(at 76.2 91.44 0)
+			(effects
+				(font
+					(size 1.27 1.27)
+				)
+				(justify left)
+			)
+		)
+		(pin "+1V8" output
+			(at 76.2 96.52 0)
+			(effects
+				(font
+					(size 1.27 1.27)
+				)
+				(justify left)
+			)
+		)
+		(pin "GND" passive
+			(at 76.2 101.6 0)
+			(effects
+				(font
+					(size 1.27 1.27)
+				)
+				(justify left)
+			)
+		)
+		(instances
+			(project "fcBoard"
+				(path "/e63e39d7-6ac0-4ffd-8aa3-1841a4541b55"
+					(page "2")
+				)
+			)
+		)
+	)
+	(sheet
+		(at 25.4 119.38)
+		(size 50.8 25.4)
+		(exclude_from_sim no)
+		(in_bom yes)
+		(on_board yes)
+		(dnp no)
+		(fields_autoplaced yes)
+		(stroke
+			(width 0.1524)
+			(type solid)
+		)
+		(fill
+			(color 194 255 194 1.0000)
+		)
+		(property "Sheetname" "USB 3.0 Hub"
+			(at 25.4 118.6684 0)
+			(effects
+				(font
+					(size 1.27 1.27)
+				)
+				(justify left bottom)
+			)
+		)
+		(property "Sheetfile" "fcBoard_USB.kicad_sch"
+			(at 25.4 145.3216 0)
+			(effects
+				(font
+					(size 1.27 1.27)
+				)
+				(justify left top)
+			)
+		)
+		(instances
+			(project "fcBoard"
+				(path "/e63e39d7-6ac0-4ffd-8aa3-1841a4541b55"
+					(page "3")
+				)
+			)
+		)
+	)
+	(sheet
+		(at 25.4 154.94)
+		(size 50.8 25.4)
+		(exclude_from_sim no)
+		(in_bom yes)
+		(on_board yes)
+		(dnp no)
+		(fields_autoplaced yes)
+		(stroke
+			(width 0.1524)
+			(type solid)
+		)
+		(fill
+			(color 194 224 255 1.0000)
+		)
+		(property "Sheetname" "Gigabit Ethernet"
+			(at 25.4 154.2284 0)
+			(effects
+				(font
+					(size 1.27 1.27)
+				)
+				(justify left bottom)
+			)
+		)
+		(property "Sheetfile" "fcBoard_Ethernet.kicad_sch"
+			(at 25.4 180.8816 0)
+			(effects
+				(font
+					(size 1.27 1.27)
+				)
+				(justify left top)
+			)
+		)
+		(instances
+			(project "fcBoard"
+				(path "/e63e39d7-6ac0-4ffd-8aa3-1841a4541b55"
+					(page "4")
+				)
+			)
+		)
+	)
+	(sheet
+		(at 25.4 190.5)
+		(size 50.8 25.4)
+		(exclude_from_sim no)
+		(in_bom yes)
+		(on_board yes)
+		(dnp no)
+		(fields_autoplaced yes)
+		(stroke
+			(width 0.1524)
+			(type solid)
+		)
+		(fill
+			(color 255 194 224 1.0000)
+		)
+		(property "Sheetname" "HDMI In/Out"
+			(at 25.4 189.7884 0)
+			(effects
+				(font
+					(size 1.27 1.27)
+				)
+				(justify left bottom)
+			)
+		)
+		(property "Sheetfile" "fcBoard_HDMI.kicad_sch"
+			(at 25.4 216.4416 0)
+			(effects
+				(font
+					(size 1.27 1.27)
+				)
+				(justify left top)
+			)
+		)
+		(instances
+			(project "fcBoard"
+				(path "/e63e39d7-6ac0-4ffd-8aa3-1841a4541b55"
+					(page "5")
+				)
+			)
+		)
+	)
+	(sheet
+		(at 25.4 226.06)
+		(size 50.8 25.4)
+		(exclude_from_sim no)
+		(in_bom yes)
+		(on_board yes)
+		(dnp no)
+		(fields_autoplaced yes)
+		(stroke
+			(width 0.1524)
+			(type solid)
+		)
+		(fill
+			(color 224 194 255 1.0000)
 		)
 		(property "Sheetname" "Peripherals"
-			(at 279.4 75.4884 0)
+			(at 25.4 225.3484 0)
 			(effects
 				(font
@@
 		)
 		(property "Sheetfile" "fcBoard_Peripherals.kicad_sch"
-			(at 279.4 107.2216 0)
-			(effects
-				(font
-					(size 1.27 1.27)
-				)
-				(justify left top)
-			)
-		)
-	)
-	(sheet
-		(at 88.9 76.2)
-		(size 50.8 30.48)
-		(exclude_from_sim no)
-		(in_bom yes)
-		(on_board yes)
-		(dnp no)
-		(fields_autoplaced yes)
-		(stroke
-			(width 0.1524)
-			(type solid)
-		)
-		(fill
-			(color 194 255 194 1.0000)
-		)
-		(property "Sheetname" "USB 3.0 Hub"
-			(at 88.9 75.4884 0)
-			(effects
-				(font
-					(size 1.27 1.27)
-				)
-				(justify left bottom)
-			)
-		)
-		(property "Sheetfile" "fcBoard_USB.kicad_sch"
-			(at 88.9 107.2216 0)
-			(effects
-				(font
-					(size 1.27 1.27)
-				)
-				(justify left top)
-			)
-		)
+			(at 25.4 252.0016 0)
+			(effects
+				(font
+					(size 1.27 1.27)
+				)
+				(justify left top)
+			)
+		)
+		(instances
+			(project "fcBoard"
+				(path "/e63e39d7-6ac0-4ffd-8aa3-1841a4541b55"
+					(page "6")
+				)
+			)
+		)
